File: ayab-shield/arduino_shield.kicad_pcb (KiCad board)
At the start: 2 copper layers, 75.1 x 53.3 mm, 35 parts, among them IC1 ULN2803A, IC2 ULN2803A, IC3 MCP2300X/P, IC4 MCP2300X/P, J1 Power, J2 Digital/PWM, J3 Analog, J4 Digital/PWM, X1 KLDX-0202-AC

Commit message: open sauce special edition
Parts:
- added G***: LOGO, LOGO, B.Cu at (146.3, 103.6)
- added kibuzzard-686AF158: G***, kibuzzard-686AF158, B.Cu at (178.1, 116.6)
- moved REF** 1.14 mm to (119.3, 82.6)
Other:
- board text added: "AYAB Shield V1.5 7/2025"
- board text removed: "AYAB-Shield V1.5 4/2025"
