File: ayab-esp32/aux-connectors.kicad_sch (KiCad schematic)
At the start: 27 parts, among them J801 AYAB_UART, J802 I2C_VBUS, J803 USER_I2C, J804 I2C_VBUS, J805 AYAB_SPI, J806 AYAB_I2C, Q801 AO3400A, Q802 AO3400A, Q803 AO3400A, Q804 AO3400A

Commit message: save in version 9
Parts:
- J801, J806: Mouser PN 855-M20-9750446 -> (none)
- J803: LCSC ID C20625577 -> C3029334; Mouser PN 485-4208 -> (none)
- J805: Mouser PN 474-GPS-00579 -> (none)
- R801, R802, R809, R810, R813, R818, R819: Mouser PN 603-RC0603JR-1347RL -> (none)
- R803, R804, R807, R808, R811, R812, R816, R817: Mouser PN 603-AC0603FR-135K1L -> (none)
- R814, R815: Mouser PN 791-RMC16K103FTP -> (none)
