File: ayab-esp32/brother-connectors.kicad_sch (KiCad schematic)
At the start: 16 parts, among them J401 900.965.CK35 SOLENOIDS A, J402 900.965.CK35 SOLENOIDS B, J403 910.950 SOLENOIDS A, J404 910.950 SOLENOIDS B, J405 910.950 ENCODERS EOL R, J406 930.940 SOLENOIDS A, J407 930.940 SOLENOIDS B, J408 910.950 EOL L, J409 930.940 EOL R, J410 930.940 ENCODERS, J411 900.965 EOL L, J412 900.965 EOL R, J413 900.965 ENCODERS, J414 930.940 EOL L

Commit message: save in version 9
Parts:
- J401: Mouser PN 538-53014-1010 -> (none)
- J402: Mouser PN 538-53014-0810 -> (none)
- J403, J405: Mouser PN 798-HNC22.5P10DS55 -> (none)
- J404: Mouser PN 798-HNC2-2.5P-8DS55 -> (none)
- J406: Mouser PN 538-22-03-5105 -> (none)
- J407: Mouser PN 538-22-03-5085 -> (none)
- J408: Mouser PN 798-HNC2-2.5P-3DS55 -> (none)
- J409, J414: footprint Library:CONN-TH_3P-P2.50_X2564WV-03-N0SN -> easyeda2kicad:CONN-TH_3P-P2.50_X2564WV-03-N0SN; Mouser PN 538-22-03-5035 -> (none)
- J410: footprint Library:CONN-TH_X2564WV-05-N0SN -> easyeda2kicad:CONN-TH_X2564WV-05-N0SN; Mouser PN 538-22-03-5055 -> (none)
- J411, J412: Mouser PN 538-53014-0310 -> (none)
- J413: Mouser PN 538-53014-0510 -> (none)
Changed lines of the file:
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@@
 			)
 		)
-		(property "Description" "Power symbol creates a global label with name \"+5V\""
+		(property "Description" ""
 			(at 55.88 102.87 0)
 			(effects
@@
 					(size 1.27 1.27)
 				)
-				(hide yes)
 			)
 		)
@@
 			)
 		)
-		(property "Footprint" "Library:CONN-TH_3P-P2.50_X2564WV-03-N0SN"
+		(property "Footprint" "easyeda2kicad:CONN-TH_3P-P2.50_X2564WV-03-N0SN"
 			(at 242.57 110.49 0)
 			(effects
@@
 					(size 1.27 1.27)
 				)
-				(hide yes)
 			)
 		)
@@
 		)
 		(property "LCSC ID" "C397419"
-			(at 242.57 110.49 0)
-			(effects
-				(font
-					(size 1.27 1.27)
-				)
-				(hide yes)
-			)
-		)
-		(property "Mouser PN" "538-22-03-5035 "
 			(at 242.57 110.49 0)
 			(effects
@@
 			)
 		)
-		(property "Description" "Power symbol creates a global label with name \"+5V\""
+		(property "Description" ""
 			(at 234.95 105.41 0)
 			(effects
@@
 					(size 1.27 1.27)
 				)
-				(hide yes)
 			)
 		)
@@
 					(size 1.27 1.27)
 				)
-				(hide yes)
 			)
 		)
@@
 		)
 		(property "LCSC ID" "C225243"
-			(at 63.5 135.89 0)
-			(effects
-				(font
-					(size 1.27 1.27)
-				)
-				(hide yes)
-			)
-		)
-		(property "Mouser PN" "538-53014-0510 "
 			(at 63.5 135.89 0)
 			(effects
@@
 					(size 1.27 1.27)
 				)
-				(hide yes)
 			)
 		)
@@
 			)
 		)
-		(property "Mouser PN" "538-53014-0310 "
-			(at 63.5 107.95 0)
-			(effects
-				(font
-					(size 1.27 1.27)
-				)
-				(hide yes)
-			)
-		)
 		(pin "1"
 		)
@@
 					(size 1.27 1.27)
 				)
-				(hide yes)
 			)
 		)
@@
 		)
 		(property "OEM" ""
-			(at 133.35 118.11 0)
-			(effects
-				(font
-					(size 1.27 1.27)
-				)
-				(hide yes)
-			)
-		)
-		(property "Mouser PN" ""
 			(at 133.35 118.11 0)
 			(effects
@@
 					(size 1.27 1.27)
 				)
-				(hide yes)
 			)
 		)
@@
 		)
 		(property "OEM" "Hirose"
-			(at 152.4 107.95 0)
-			(effects
-				(font
-					(size 1.27 1.27)
-				)
-				(hide yes)
-			)
-		)
-		(property "Mouser PN" "798-HNC2-2.5P-3DS55 "
 			(at 152.4 107.95 0)
 			(effects
@@
 					(size 1.27 1.27)
 				)
-				(hide yes)
 			)
 		)
@@
 		)
 		(property "OEM" "Hirose"
-			(at 152.4 77.47 0)
-			(effects
-				(font
-					(size 1.27 1.27)
-				)
-				(hide yes)
-			)
-		)
-		(property "Mouser PN" "798-HNC2-2.5P-8DS55 "
 			(at 152.4 77.47 0)
 			(effects
@@
 			)
 		)
-		(property "Description" "Power symbol creates a global label with name \"+12V\""
+		(property "Description" ""
 			(at 144.78 34.29 0)
 			(effects
@@
 					(size 1.27 1.27)
 				)
-				(hide yes)
 			)
 		)
@@
 					(size 1.27 1.27)
 				)
-				(hide yes)
 			)
 		)
@@
 		)
 		(property "OEM" "HR(Joint Tech Elec)"
-			(at 242.57 52.07 0)
-			(effects
-				(font
-					(size 1.27 1.27)
-				)
-				(hide yes)
-			)
-		)
-		(property "Mouser PN" "538-22-03-5105 "
 			(at 242.57 52.07 0)
 			(effects
@@
 			)
 		)
-		(property "Description" "Power symbol creates a global label with name \"GND\" , ground"
+		(property "Description" ""
 			(at 53.34 144.78 0)
 			(effects
@@
 					(size 1.27 1.27)
 				)
-				(hide yes)
 			)
 		)
@@
 					(size 1.27 1.27)
 				)
-				(hide yes)
 			)
 		)
@@
 		)
 		(property "OEM" ""
-			(at 133.35 120.65 0)
-			(effects
-				(font
-					(size 1.27 1.27)
-				)
-				(hide yes)
-			)
-		)
-		(property "Mouser PN" ""
 			(at 133.35 120.65 0)
 			(effects
@@
 			)
 		)
-		(property "Description" "Power symbol creates a global label with name \"+12V\""
+		(property "Description" ""
 			(at 234.95 36.83 0)
 			(effects
@@
 					(size 1.27 1.27)
 				)
-				(hide yes)
 			)
 		)
@@
 					(size 1.27 1.27)
 				)
-				(hide yes)
 			)
 		)
@@
 		)
 		(property "OEM" "Hirose"
-			(at 152.4 49.53 0)
-			(effects
-				(font
-					(size 1.27 1.27)
-				)
-				(hide yes)
-			)
-		)
-		(property "Mouser PN" "798-HNC22.5P10DS55 "
 			(at 152.4 49.53 0)
 			(effects
@@
 					(size 1.27 1.27)
 				)
-				(hide yes)
 			)
 		)
@@
 		)
 		(property "LCSC ID" "C225246"
-			(at 63.5 77.47 0)
-			(effects
-				(font
-					(size 1.27 1.27)
-				)
-				(hide yes)
-			)
-		)
-		(property "Mouser PN" "538-53014-0810 "
 			(at 63.5 77.47 0)
 			(effects
@@
 			)
 		)
-		(property "Description" "Power symbol creates a global label with name \"+12V\""
+		(property "Description" ""
 			(at 55.88 34.29 0)
 			(effects
@@
 					(size 1.27 1.27)
 				)
-				(hide yes)
 			)
 		)
@@
 					(size 1.27 1.27)
 				)
-				(hide yes)
 			)
 		)
@@
 		)
 		(property "LCSC ID" "C476906"
-			(at 242.57 80.01 0)
-			(effects
-				(font
-					(size 1.27 1.27)
-				)
-				(hide yes)
-			)
-		)
-		(property "Mouser PN" "538-22-03-5085 "
 			(at 242.57 80.01 0)
 			(effects
@@
 			)
 		)
-		(property "Description" "Power symbol creates a global label with name \"GND\" , ground"
+		(property "Description" ""
 			(at 143.51 144.78 0)
 			(effects
@@
 					(size 1.27 1.27)
 				)
-				(hide yes)
 			)
 		)
@@
 					(size 1.27 1.27)
 				)
-				(hide yes)
 			)
 		)
@@
 			)
 		)
-		(property "Mouser PN" "798-HNC22.5P10DS55 "
-			(at 152.4 130.81 0)
-			(effects
-				(font
-					(size 1.27 1.27)
-				)
-				(hide yes)
-			)
-		)
 		(pin "1"
 		)
@@
 			)
 		)
-		(property "Description" "Power symbol creates a global label with name \"+5V\""
+		(property "Description" ""
 			(at 140.97 101.6 0)
 			(effects
@@
 					(size 1.27 1.27)
 				)
-				(hide yes)
 			)
 		)
@@
 					(size 1.27 1.27)
 				)
-				(hide yes)
 			)
 		)
@@
 		)
 		(property "LCSC ID" "C2834606"
-			(at 63.5 49.53 0)
-			(effects
-				(font
-					(size 1.27 1.27)
-				)
-				(hide yes)
-			)
-		)
-		(property "Mouser PN" "538-53014-1010 "
 			(at 63.5 49.53 0)
 			(effects
@@
 			)
 		)
-		(property "Footprint" "Library:CONN-TH_X2564WV-05-N0SN"
+		(property "Footprint" "easyeda2kicad:CONN-TH_X2564WV-05-N0SN"
 			(at 242.57 138.43 0)
 			(effects
@@
 					(size 1.27 1.27)
 				)
-				(hide yes)
 			)
 		)
@@
 		)
 		(property "LCSC ID" "C707030"
-			(at 242.57 138.43 0)
-			(effects
-				(font
-					(size 1.27 1.27)
-				)
-				(hide yes)
-			)
-		)
-		(property "Mouser PN" "538-22-03-5055 "
 			(at 242.57 138.43 0)
 			(effects
@@
 			)
 		)
-		(property "Description" "Power symbol creates a global label with name \"GND\" , ground"
+		(property "Description" ""
 			(at 232.41 147.32 0)
 			(effects
@@
 					(size 1.27 1.27)
 				)
-				(hide yes)
 			)
 		)
@@
 					(size 1.27 1.27)
 				)
-				(hide yes)
 			)
 		)
@@
 		)
 		(property "LCSC ID" "C225241"
-			(at 63.5 120.65 0)
-			(effects
-				(font
-					(size 1.27 1.27)
-				)
-				(hide yes)
-			)
-		)
-		(property "Mouser PN" "538-53014-0310 "
 			(at 63.5 120.65 0)
 			(effects
@@
 			)
 		)
-		(property "Footprint" "Library:CONN-TH_3P-P2.50_X2564WV-03-N0SN"
+		(property "Footprint" "easyeda2kicad:CONN-TH_3P-P2.50_X2564WV-03-N0SN"
 			(at 242.57 123.19 0)
 			(effects
@@
 					(size 1.27 1.27)
 				)
-				(hide yes)
 			)
 		)
@@
 			(at 242.57 123.19 0)
 			(effects
-				(font
-					(size 1.27 1.27)
-				)
-				(hide yes)
-			)
-		)
-		(property "Mouser PN" "538-22-03-5035 "
-			(at 242.57 123.19 0)
-			(effects
