File: ayab-esp32/ioconditioning.kicad_sch (KiCad schematic)
At the start: 45 parts, among them J701 CTRL_3v3, J702 CTRL_5V, U701 SN74LVC4245, U702 LM393, U703 LM393

Commit message: save in version 9
Parts:
- C701, C702, C703, C704: Mouser PN 187-CL10B104MB8NNNC -> (none)
- J701, J702: Mouser PN 649-67997-108HLF -> (none)
- R701, R702, R703, R704, R705, R706, R707, R708, R709, R710, R711, R712, R713, R714, R719, R720, R721, R722: Mouser PN 791-RMC16K103FTP -> (none)
- R715, R716, R717, R718: Mouser PN 71-CRCW0603100KJNEAC -> (none)
- R723, R725, R728, R730: Mouser PN 71-CRCW06034K70FKEAC -> (none)
- R724, R726: Mouser PN 71-CRCW06031K24FKEAC -> (none)
- R727, R729: Mouser PN 603-RC0603FR-073K3P -> (none)
- R731, R732: Mouser PN 603-RC0603JR-0722KL -> (none)
- R733, R734: Mouser PN 603-AC0603FR-1047KL -> (none)
- U701: Mouser PN 595-SN74LVC4245APWRG -> (none)
- U702, U703: Mouser PN 926-LM393M/NOPB -> (none)
