File: ayab-esp32/mcu.kicad_sch (KiCad schematic)
At the start: 27 parts, among them J201 SPARE1, J202 SPARE0, Q201 AO3400A, SW201 USER, SW202 RESET, SW203 BOOTSEL, U201 ESP32-S3-MINI-1

Commit message: save in version 9
Parts:
- added TP1: ADC0, symbol Connector:TestPoint
- added TP2: ADC1, symbol Connector:TestPoint
- BUZZER201: footprint Library:BUZ-SMD_4P-L8.5-W8.5-P8.50-BR -> easyeda2kicad:BUZ-SMD_4P-L8.5-W8.5-P8.50-BR; Mouser PN 179-CMT-8504-99SMTTR -> (none)
- C201, C202, C203, C204: Mouser PN 187-CL10B104MB8NNNC -> (none)
- C205: Mouser PN 963-TMK212BBJ106KG-T -> (none)
- D201: Mouser PN 755-SML-H12Y8TT86C -> (none)
- D202: Mouser PN 749-SM0805PGC -> (none)
- D203: Mouser PN 749-SM0805RC -> (none)
- D204: Mouser PN 750-SS54B-HF -> (none)
- J201, J202: Mouser PN 855-M20-9750446 -> (none)
- R201, R205, R206, R207, R208, R211: Mouser PN 791-RMC16K103FTP -> (none)
- R202, R203: Mouser PN 603-AC0603FR-135K1L -> (none)
- R204: value 10k -> 5k1; LCSC ID C25804 -> C23186; Mouser PN 603-AC0603FR-135K1L -> (none)
- R212: Mouser PN 71-CRCW06030000Z0EC -> (none)
- SW201, SW202, SW203: footprint Library:KEY-TH_4P-L7.5-W11.5-P4.5 -> easyeda2kicad:KEY-TH_4P-L7.5-W11.5-P4.5
- U201: footprint Library:ESP32-S3-MINI-1 -> Espressif:ESP32-S3-MINI-1; Mouser PN 356-ESP32-S3-MINI1N8 -> (none)
Connections:
- net EOL_L_N: no longer names the net of U201.6 (GPIO2/TOUCH2/ADC1_CH1)
- net EOL_L_N: now also TP1.1
- net EOL_L_P renamed EOL_L
- net EOL_R_N: no longer names the net of U201.8 (GPIO4/TOUCH4/ADC1_CH3)
- net EOL_R_N: now also TP2.1
- net EOL_R_P renamed EOL_R
