File: ayab-esp32/psu.kicad_sch (KiCad schematic)
At the start: 47 parts, among them J601 VIN, J602 Brother_5P, J604 Brother_4R, Q601 LP9435LT1G, U601 XL1509, U602 XL1509

Commit message: save in version 9
Parts:
- removed Q601: LP9435LT1G, Package_TO_SOT_SMD:SOT-23, symbol ayab-lib:AO3401A
- removed R601: 10k, Resistor_SMD:R_0603_1608Metric, symbol ayab-lib:R_Small_US
- C601, C602, C603, C604, C605, C610, C611, C616, C617, C618, C619, C620, C621: Mouser PN 963-TMK212BBJ106KG-T -> (none)
- C606, C607, C609, C612, C613: Mouser PN 661-EMZR250ARA221MF8 -> (none)
- C614, C615: Mouser PN 80-C0603C332K2RACTU -> (none)
- D601: footprint Library:MBF-SMD_L4.8-W3.8-P2.54-LS6.8-TL -> easyeda2kicad:MBF-SMD_L4.8-W3.8-P2.54-LS6.8-TL
- D602, D603, D604: Mouser PN 696-SML-LXT0805IW -> (none)
- D605, D606: Mouser PN 750-SS54B-HF -> (none)
- J601: footprint Library:DC-IN-TH_DC-005-5A-2.0-SMT -> easyeda2kicad:DC-IN-TH_DC-005-5A-2.0-SMT; Mouser PN 806-KLDXSMT20202BT -> (none)
- L601, L602: Mouser PN 580-49470SC -> (none)
- R603: Mouser PN 791-RMC16K103FTP -> (none)
- R604: Mouser PN 603-AC0603FR-135K1L -> (none)
- R605, R608: Mouser PN 603-RC0603FR-073K3P -> (none)
- R606, R607: Mouser PN 71-CRCW06031K24FKEAC -> (none)
- R609: Mouser PN 279-CRG0603F1K8 -> (none)
- R610, R611: footprint Resistor_SMD:R_0805_2012Metric -> Resistor_SMD:R_0603_1608Metric; LCSC ID C17477 -> C21189; Mouser PN 71-CRCW06030000Z0EC -> (none)
- U601, U602: LCSC ID C74192 -> C74193
Connections:
- net 12V: now also D601.3 (+); no longer D601.1 (+)
- net 5V_SW: now also R611.1
- net GND: now also D601.4 (-); no longer D601.2 (-)
- net INP_1: now also D601.1; no longer D601.3
- net INP_2: now also D601.2; no longer D601.4
Other:
- moved on the sheet: R611, TP602
